Commit message: Robot can make moves

File: ros2_ws/src/ur_tcp_moveit_config/srdf/ur_macro.srdf.xacro (robot description, xacro)
@@ -27,4 +27,20 @@
         <joint name="wrist_3_joint" value="0"/>
     </group_state>
+    <group_state name="idle" group="ur_manipulator">
+        <joint name="elbow_joint" value="0.79"/>
+        <joint name="shoulder_lift_joint" value="-1.57"/>
+        <joint name="shoulder_pan_joint" value="1.57"/>
+        <joint name="wrist_1_joint" value="-1.57"/>
+        <joint name="wrist_2_joint" value="-1.57"/>
+        <joint name="wrist_3_joint" value="0"/>
+    </group_state>
+    <group_state name="out" group="ur_manipulator">
+        <joint name="elbow_joint" value="1.94"/>
+        <joint name="shoulder_lift_joint" value="-1.36"/>
+        <joint name="shoulder_pan_joint" value="2.27"/>
+        <joint name="wrist_1_joint" value="-2.15"/>
+        <joint name="wrist_2_joint" value="-1.57"/>
+        <joint name="wrist_3_joint" value="0.7"/>
+    </group_state>
     <!--DISABLE COLLISIONS: By default it is assumed that any link of the robot could potentially come into collision with any other link in the robot. This tag disables collision checking between a specified pair of links. -->
     <disable_collisions link1="base_link_inertia" link2="ground_plane" reason="Adjacent"/>

Commit message: Some fixes

File: ros2_ws/src/ur_tcp_moveit_config/srdf/ur_macro.srdf.xacro (robot description, xacro)
@@ -36,9 +36,9 @@
     </group_state>
     <group_state name="out" group="ur_manipulator">
-        <joint name="elbow_joint" value="1.94"/>
-        <joint name="shoulder_lift_joint" value="-1.36"/>
+        <joint name="elbow_joint" value="1.48"/>
+        <joint name="shoulder_lift_joint" value="-1.5"/>
         <joint name="shoulder_pan_joint" value="2.27"/>
-        <joint name="wrist_1_joint" value="-2.15"/>
-        <joint name="wrist_2_joint" value="-1.57"/>
+        <joint name="wrist_1_joint" value="-1.57"/>
+        <joint name="wrist_2_joint" value="-1.5 7"/>
         <joint name="wrist_3_joint" value="0.7"/>
     </group_state>

Commit message: Robot working

File: ros2_ws/src/ur_tcp_moveit_config/srdf/ur_macro.srdf.xacro (robot description, xacro)
@@ -28,9 +28,9 @@
     </group_state>
     <group_state name="idle" group="ur_manipulator">
-        <joint name="elbow_joint" value="0.79"/>
-        <joint name="shoulder_lift_joint" value="-1.57"/>
+        <joint name="elbow_joint" value="0"/>
+        <joint name="shoulder_lift_joint" value="-1.4927"/>
         <joint name="shoulder_pan_joint" value="1.57"/>
-        <joint name="wrist_1_joint" value="-1.57"/>
-        <joint name="wrist_2_joint" value="-1.57"/>
+        <joint name="wrist_1_joint" value="-1.5621"/>
+        <joint name="wrist_2_joint" value="0"/>
         <joint name="wrist_3_joint" value="0"/>
     </group_state>
@@ -40,5 +40,5 @@
         <joint name="shoulder_pan_joint" value="2.27"/>
         <joint name="wrist_1_joint" value="-1.57"/>
-        <joint name="wrist_2_joint" value="-1.5 7"/>
+        <joint name="wrist_2_joint" value="-1.57"/>
         <joint name="wrist_3_joint" value="0.7"/>
     </group_state>
