Commit message: Change vertical move to 10cm to avoid collisions with pieces

File: ros2_ws/src/ur3_tcp/urdf/gripper_dummy.xacro (robot description, xacro)
@@ -7,6 +7,6 @@
     <!-- ==================== PARAMETERS ==================== -->
     <xacro:property name="sphere_radius" value="0.01"/> <!-- 1 cm radius -->
-    <xacro:property name="gripper_radius" value="0.05"/> <!-- 1 cm radius -->
-    <xacro:property name="gripper_length" value="0.06"/> <!-- 1 cm radius -->
+    <xacro:property name="gripper_radius" value="0.06"/> <!-- 1 cm radius -->
+    <xacro:property name="gripper_length" value="0.08"/> <!-- 1 cm radius -->
     <xacro:property name="sphere_color_orange" value="1.0 0.5 0.0 1.0"/> <!-- Orange RGBA -->
     <xacro:property name="sphere_color_green" value="0.3 1.0 0.3 1.0"/> <!-- green RGBA -->
@@ -14,8 +14,11 @@
     <link name="${prefix}_gripper_dummy">
       <visual>
-      <origin xyz="0 0 0.06" rpy="${offset_rpy}"/>
+      <origin xyz="0 0 ${gripper_length/2}" rpy="${offset_rpy}"/>
         <geometry>
           <sphere radius="${sphere_radius}"/>
         </geometry>
+        <!-- <geometry>
+          <cylinder radius="${gripper_radius}" length="${gripper_length}"/>
+        </geometry> -->
         <material name="green">
           <color rgba="${sphere_color_green}"/>

Commit message: Add promotion move, game beetween two robots

File: ros2_ws/src/ur3_tcp/urdf/gripper_dummy.xacro (robot description, xacro)
@@ -6,7 +6,8 @@
   <xacro:macro name="gripper_dummy" params="prefix parent_link offset_xyz:='0 0 0' offset_rpy:='0 0 0'">
     <!-- ==================== PARAMETERS ==================== -->
-    <xacro:property name="sphere_radius" value="0.01"/> <!-- 1 cm radius -->
+    <xacro:property name="sphere_radius" value="0.0175"/> <!-- 1 cm radius -->
     <xacro:property name="gripper_radius" value="0.06"/> <!-- 1 cm radius -->
-    <xacro:property name="gripper_length" value="0.08"/> <!-- 1 cm radius -->
+    <xacro:property name="gripper_length" value="0.14"/> <!-- 1 cm radius -->
+    <xacro:property name="gripper_colisions_length" value="0.1"/>
     <xacro:property name="sphere_color_orange" value="1.0 0.5 0.0 1.0"/> <!-- Orange RGBA -->
     <xacro:property name="sphere_color_green" value="0.3 1.0 0.3 1.0"/> <!-- green RGBA -->

Commit message: Minor imporvements

File: ros2_ws/src/ur3_tcp/urdf/gripper_dummy.xacro (robot description, xacro)
@@ -8,5 +8,5 @@
     <xacro:property name="sphere_radius" value="0.0175"/> <!-- 1 cm radius -->
     <xacro:property name="gripper_radius" value="0.06"/> <!-- 1 cm radius -->
-    <xacro:property name="gripper_length" value="0.14"/> <!-- 1 cm radius -->
+    <xacro:property name="gripper_length" value="0.167"/> <!-- 1 cm radius -->
     <xacro:property name="gripper_colisions_length" value="0.1"/>
     <xacro:property name="sphere_color_orange" value="1.0 0.5 0.0 1.0"/> <!-- Orange RGBA -->
